File: espdisplay.kicad_pcb (KiCad board)
At the start: 2 copper layers, 34.3 x 30 mm, 11 parts, among them J1 PWR, J2 UReg, J3 DOut, J4 Serial, J5 IO32, SW1 RESET, SW2 BOOT, U1 ESP-WROOM-32

Commit message: Rev A2
Other:
- board text added: "Rev A2"
- board text removed: "Rev A1"
Changed lines of the file:
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@@
     (links 28)
     (no_connects 0)
-    (area 147.553499 92.009999 181.993501 122.132001)
+    (area 143.5945 83.49 185.862 122.132001)
     (thickness 1.6)
     (drawings 38)
@@
     (descr "JST PH series connector, S2B-PH-K, side entry type, through hole, Datasheet: http://www.jst-mfg.com/product/pdf/eng/ePH.pdf")
     (tags "connector jst ph")
-    (fp_text reference J1 (at -2.667 2.667 360) (layer F.SilkS)
+    (fp_text reference J1 (at -2.5908 2.667 360) (layer F.SilkS)
       (effects (font (size 1 1) (thickness 0.15)))
     )
@@
     (effects (font (size 0.7 0.7) (thickness 0.15)) (justify mirror))
   )
-  (gr_text GND (at 152.0195 92.9735) (layer F.SilkS)
+  (gr_text GND (at 152.0195 93.0497) (layer F.SilkS)
     (effects (font (size 1 1) (thickness 0.15)))
   )
-  (gr_text "Rev A1" (at 149.9145 121.168) (layer F.SilkS)
+  (gr_text "Rev A2" (at 149.9145 121.168) (layer F.SilkS)
     (effects (font (size 0.7 0.7) (thickness 0.12)))
   )
